File: kicad/midi_decoder.kicad_pcb (KiCad board)
At the start: 2 copper layers, 152.3 x 128.5 mm, 174 parts, among them J10 Modulation CV, J11 CAN, J12 Bus Connector, J13 bus (board), J14 MIDI, J15 bus (controller), J2 MIDI, J3 MIDI IN, J4 MIDI THRU, J5 Note 1, J6 Gate 1, J7 Note 2, J8 Gate 2, J9 Expression CV, P1 Spacer 2M without hole, P10 3.5mm single channel, P11 3.5mm single channel, P12 3.5mm single channel, P13 3.5mm single channel, P14 3.5mm single channel, P15 3.5mm single channel, P2 Spacer 2M without hole, P3 Spacer 2M without hole, P4 LED Window 5mm, P5 LED Window 5mm, P6 PEL12D, P7 Spacer 2M without hole, P8 DIN 5 pin, P9 DIN 5 pin, Q1 MMBT3906, Q2 MMBT3906, Q3 MMBT3906, Q4 MMBT3904, Q5 MMBT3904, Q6 MMBT3904, Q7 MMBT3904, SW1 Reset, U1 PEL12D-4225S-S2024, U10 TL074, U11 CD4052B, U12 REF3030, U13 MCP4011-103E/SN, U2 6N138, U3 SN65HVD1050D, U4 MCP4011-503E/SN, U5 TL074, U6 MCP4011-503E/SN, U7 MCP4011-103E/SN, U9 TL074, Y1 ECS-240-9

Commit message: revision 1
Parts:
- removed the C11 at (112.3, 144.2)
- removed the C12 at (130.1, 149.6)
- removed the C15 at (104.7, 124.3)
- removed the C17 at (100.4, 129.3)
- removed NT2: NetTie_2, NetTie:NetTie-2_SMD_Pad0.5mm
- removed the R34 at (93.6, 98.7)
- removed the R39 at (100.4, 131.6)
- removed the R42 at (104.6, 122.1)
- removed the R45 at (100.6, 124.3)
- removed the U11 at (102.5, 142.6)
- removed the U6 at (128.2, 145.2)
- removed Y1: ECS-240-9, Crystal:Crystal_SMD_3225-4Pin_3.2x2.5mm_HandSoldering
- added C14: 4.7u tantal, Capacitor_Tantalum_SMD:CP_EIA-3216-10_Kemet-I_Pad1.58x1.35mm_HandSolder, F.Cu at (121.8, 128.2)
- added C16: 100u, Capacitor_SMD:CP_Elec_5x5.3, F.Cu at (151.5, 133.0)
- added C18: 100u, Capacitor_THT:CP_Radial_D6.3mm_P2.50mm, F.Cu at (152.0, 138.5)
- added C21: 4.7u tantal, Capacitor_Tantalum_SMD:CP_EIA-3216-10_Kemet-I_Pad1.58x1.35mm_HandSolder, F.Cu at (121.6, 146.8)
- added C22: 100u, Capacitor_THT:CP_Radial_D6.3mm_P2.50mm, F.Cu at (152.0, 145.5)
- added C26: 56p, Capacitor_SMD:C_0805_2012Metric_Pad1.18x1.45mm_HandSolder, B.Cu at (89.5, 104.8)
- added C31: 0.1u, Capacitor_SMD:C_0805_2012Metric_Pad1.18x1.45mm_HandSolder, B.Cu at (93.5, 124.7)
- added C32: 0.1u, Capacitor_SMD:C_0805_2012Metric_Pad1.18x1.45mm_HandSolder, B.Cu at (91.5, 126.0)
- added C37: 56p, Capacitor_SMD:C_0805_2012Metric_Pad1.18x1.45mm_HandSolder, B.Cu at (136.5, 137.3)
- added C38: 56p, Capacitor_SMD:C_0805_2012Metric_Pad1.18x1.45mm_HandSolder, B.Cu at (139.5, 137.2)
- added C9: 0.1u, Capacitor_SMD:C_0805_2012Metric_Pad1.18x1.45mm_HandSolder, F.Cu at (121.0, 132.0)
- added D5: 1N4448WS, Diode_SMD:D_SOD-323_HandSoldering, F.Cu at (86.0, 132.0)
- added D6: 1N4448WS, Diode_SMD:D_SOD-323_HandSoldering, F.Cu at (108.8, 132.8)
- added D7: 1N4448WS, Diode_SMD:D_SOD-323_HandSoldering, F.Cu at (108.8, 145.5)
- added L1: 22u, Inductor_SMD:L_0805_2012Metric_Pad1.05x1.20mm_HandSolder, F.Cu at (146.5, 129.8)
- added Q1: BC847B, Package_TO_SOT_SMD:SOT-23, F.Cu at (76.0, 48.8)
- added Q10: MMBFJ176, Package_TO_SOT_SMD:SOT-23, F.Cu at (135.1, 128.6)
- added Q11: MMBFJ176, Package_TO_SOT_SMD:SOT-23, F.Cu at (143.6, 128.3)
- added Q12: MMBFJ112, Package_TO_SOT_SMD:SOT-23, F.Cu at (108.8, 148.6)
- added Q13: BC847B, Package_TO_SOT_SMD:SOT-23, B.Cu at (88.9, 55.3)
- added Q15: BC847B, Package_TO_SOT_SMD:SOT-23, B.Cu at (73.4, 49.0)
- added Q16: BC847B, Package_TO_SOT_SMD:SOT-23, B.Cu at (88.8, 59.0)
- added Q18: BC847B, Package_TO_SOT_SMD:SOT-23, B.Cu at (67.8, 44.2)
- added Q2: BC847B, Package_TO_SOT_SMD:SOT-23, F.Cu at (85.8, 48.8)
- added Q8: BC857B, Package_TO_SOT_SMD:SOT-23, F.Cu at (104.2, 125.3)
- added Q9: MMBFJ112, Package_TO_SOT_SMD:SOT-23, F.Cu at (108.8, 129.8)
- added R2: 10k, Diode_SMD:D_0805_2012Metric_Pad1.15x1.40mm_HandSolder, F.Cu at (76.0, 51.8)
- added R22: 806k 1%, Diode_SMD:D_0805_2012Metric_Pad1.15x1.40mm_HandSolder, F.Cu at (94.5, 108.5)
- added R28: 220k, Diode_SMD:D_0805_2012Metric_Pad1.15x1.40mm_HandSolder, F.Cu at (77.5, 136.8)
- added R40: 220k, Diode_SMD:D_0805_2012Metric_Pad1.15x1.40mm_HandSolder, F.Cu at (104.2, 122.2)
- added R43: 470k, Resistor_SMD:R_0805_2012Metric_Pad1.20x1.40mm_HandSolder, F.Cu at (135.0, 131.8)
- added R47: 22k, Resistor_SMD:R_0805_2012Metric_Pad1.20x1.40mm_HandSolder, F.Cu at (131.8, 127.8)
- added R54: 100k, Resistor_SMD:R_0805_2012Metric_Pad1.20x1.40mm_HandSolder, F.Cu at (131.8, 131.8)
- added R55: 100k, Resistor_SMD:R_0805_2012Metric_Pad1.20x1.40mm_HandSolder, F.Cu at (140.5, 132.0)
- added R57: 470k, Resistor_SMD:R_0805_2012Metric_Pad1.20x1.40mm_HandSolder, F.Cu at (143.5, 132.0)
- added R58: 22k, Resistor_SMD:R_0805_2012Metric_Pad1.20x1.40mm_HandSolder, F.Cu at (140.5, 128.0)
- added R64: 220k, Diode_SMD:D_0805_2012Metric_Pad1.15x1.40mm_HandSolder, B.Cu at (91.0, 62.2)
- added R72: 22k, Diode_SMD:D_0805_2012Metric_Pad1.15x1.40mm_HandSolder, B.Cu at (75.8, 52.0)
- added R74: 47k, Diode_SMD:D_0805_2012Metric_Pad1.15x1.40mm_HandSolder, B.Cu at (87.0, 62.2)
- added U14: MCP4011-503E/SN, Package_SO:SOIC-8_3.9x4.9mm_P1.27mm, F.Cu at (114.8, 148.8)
- added U8: TL072, Package_SO:SOIC-8_3.9x4.9mm_P1.27mm, F.Cu at (92.5, 126.4)
- added U9: MCP4011-503E/SN, Package_SO:SOIC-8_3.9x4.9mm_P1.27mm, F.Cu at (114.8, 130.2)
- added XTAL1: ABM7-24.000MHZ-D2Y-T, MyCrystal:XTAL_ABM7_ABR_handsoldering, B.Cu at (141.1, 94.0)
- C17: renamed from C26; value 0.1u -> 100u; footprint Capacitor_SMD:C_0805_2012Metric_Pad1.18x1.45mm_HandSolder -> Capacitor_SMD:CP_Elec_5x5.3; moved to F.Cu
- C24: renamed from C29; value 8p -> 18p
- C25: renamed from C27; value 8p -> 18p
- C28: renamed from C13; moved to B.Cu
- C30: renamed from C16; moved to B.Cu
- C33: renamed from C3; moved to B.Cu
- C36: renamed from C23; moved to B.Cu
- D1: value Note 2 -> Note 1
- D4: value 1N4148 -> 1N4448WS; footprint Diode_THT:D_DO-35_SOD27_P7.62mm_Horizontal -> Diode_SMD:D_SOD-323_HandSoldering
- MB1: renamed from mouse-bite-2mm-slot; value VAL** -> MB1
- MB2: renamed from mouse-bite-2mm-slot; value VAL** -> MB2
- MB3: renamed from mouse-bite-2mm-slot; value VAL** -> mb3
- MB4: renamed from mouse-bite-2mm-slot; value VAL** -> MB4
- MB5: renamed from mouse-bite-2mm-slot; value VAL** -> MB5
- Q14: renamed from Q6; value MMBT3904 -> BC847B
- Q17: renamed from Q7; value MMBT3904 -> BC847B
- Q3: renamed from Q1; value MMBT3906 -> BC857B
- Q4: renamed from Q2; value MMBT3906 -> BC857B
- Q5: renamed from Q4; value MMBT3904 -> BC847B
- Q6: renamed from Q3; value MMBT3906 -> BC857B
- Q7: renamed from Q5; value MMBT3904 -> BC847B
- R14: renamed from R63; value 10k -> 22k; moved to F.Cu
- R17: renamed from R38; value 10k -> 100k
- R20: renamed from R37; value 10k -> 22k
- R23: renamed from R43; value 470k -> 470k 1%
- R24: renamed from R41; value 470k -> 500k 1%
- R26: renamed from R36; value 1meg -> 220k
- R27: renamed from R55; value 150k 1% -> 200k 0.1%
- R3: renamed from R2; value 1k -> 10k
- R31: renamed from R48; value 145k 1% -> 200k 0.1%
- R32: renamed from R54; value 145k -> 95.3k
- R33: renamed from R49; value 145k 1% -> 200k 0.1%
- R35: renamed from R40; value 10k -> 10k 1%
- R36: renamed from R47; value 4.7meg -> 10k
- R37: renamed from R46; value 10k -> 10k 1%
- R38: renamed from R44; value 10k -> 10k 1%
- R41: renamed from R53; value 145k -> 95.3k
- R42: renamed from R51; value 150k 1% -> 200k 0.1%
- R44: renamed from R28; value 330k -> 470k
- R45: renamed from R32; value 270k -> 200k
- R52: renamed from R33; value 470k -> 200k; footprint Diode_SMD:D_0805_2012Metric_Pad1.15x1.40mm_HandSolder -> Resistor_SMD:R_0805_2012Metric_Pad1.20x1.40mm_HandSolder
- R56: renamed from R35; value 1meg -> 470k; footprint Diode_SMD:D_0805_2012Metric_Pad1.15x1.40mm_HandSolder -> Resistor_SMD:R_0805_2012Metric_Pad1.20x1.40mm_HandSolder
- R6: renamed from R9; value 1k -> 2.2k
- R60: renamed from R31; value 200k -> 100k
- R63: renamed from R18; value 200k -> 100k
- R69: renamed from R5; value 10k -> 2.2k; moved to B.Cu
- R7: renamed from R8; value 220 -> 2.2k
- R71: renamed from R3; value 220 -> 2.2k; moved to B.Cu
- R73: renamed from R6; value 10k -> 220k; moved to B.Cu
- R77: renamed from R73; value 10k -> 47k
- R83: renamed from R20; value 330k -> 5; moved to B.Cu
- R84: renamed from R21; value 270k -> 5; moved to B.Cu
- U10: renamed from U9; value TL074 -> LMV324A
- U6: renamed from U4; value MCP4011-503E/SN -> DG419LDY
- moved C33 65.4 mm to (80.5, 130.5), turned to -90 degrees
- moved C17 62.4 mm to (151.5, 127.0), turned to 0 degrees
- moved U6 62.1 mm to (80.2, 131.3)
- moved R56 59.2 mm to (143.5, 136.2)
- moved R52 49.1 mm to (138.8, 121.5), turned to -90 degrees
- moved U10 47.7 mm to (114.8, 139.2)
- moved R34 39.3 mm to (97.5, 127.8), turned to 90 degrees
- moved R41 37.9 mm to (95.0, 131.8), turned to 90 degrees
- moved R17 37.2 mm to (86.0, 97.0), turned to 90 degrees
- moved Q7 36.8 mm to (94.2, 97.1)
- moved D4 36.3 mm to (90.8, 97.0)
- moved U12 36.2 mm to (100.3, 142.6)
- moved U5 34.7 mm to (94.7, 112.8), turned to 90 degrees
- moved C36 34.2 mm to (100.5, 144.5), turned to -90 degrees
- moved R20 34.1 mm to (88.2, 97.0), turned to 90 degrees
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- renumbered C22 to C1, C1 to C11, C7 to C12, C6 to C13, C5 to C15, C2 to C19, C21 to C2, C31 to C23, C24 to C27, C25 to C29, C18 to C3, C30 to C34, C28 to C35, C14 to C4, C8 to C5, C19 to C6, C9 to C7, C4 to C8, D3 to D2, D2 to D3, H2 to H1, H1 to H2, J4 to J1, J8 to J10, J10 to J12, J12 to J13, J15 to J14, J3 to J2, J2 to J3, J14 to J4, J13 to J6, J6 to J8, P5 to P1, P14 to P10, P15 to P11, P9 to P12, P2 to P13, P1 to P14, P3 to P15, P7 to P16, P4 to P2, REF** to P3, P6 to P4, P11 to P5, P10 to P6, P8 to P7, P12 to P8, P13 to P9, R14 to R11, R16 to R12, R15 to R13, R7 to R15, R59 to R16, R56 to R18, R57 to R19, R58 to R21, R60 to R25, R50 to R29, R61 to R30, R52 to R34, R29 to R39, R27 to R46, R26 to R48, R25 to R49, R13 to R5, R24 to R50, R23 to R51, R30 to R53, R19 to R59, R22 to R61, R17 to R62, R62 to R65, R67 to R66, R64 to R67, R65 to R68, R74 to R70, R72 to R75, R66 to R76, R75 to R78, R68 to R79, R11 to R8, R69 to R80, R70 to R81, R71 to R82, R12 to R9, U3 to U11, U13 to U12, U5 to U13, U10 to U3, U8 to U4, U12 to U5
Connections:
- C17 pad 1: GND -> +5V
- C17 pad 2: -12V -> GND
- C20 pad 1: +5V -> GND
- C20 pad 2: DGND -> +A5V
- C27 pad 1: +12V -> +A12V
- C28 pad 2: -12V -> -A12V
- C29 pad 1: +12V -> +A5V
- C30 pad 1: DGND -> GND
- C30 pad 2: +5V -> +A5V
- C33 pad 1: DGND -> +A12V
- C33 pad 2: +5V -> GND
- C34 pad 1: +12V -> +A12V
- C35 pad 2: -12V -> -A12V
- C36 pad 1: DGND -> GND
- C36 pad 2: +5V -> +A5V
- C5 pad 2: Net-(C10-Pad2) (its old number) -> Net-(U10A-+)
- C8 pad 2: Net-(C15-Pad2) (its old number) -> Net-(U10B-+)
- D1 pad 1: Net-(D4-K1) -> Net-(D1-K1)
- D1 pad 3: Net-(D4-K2) -> Net-(D1-K2)
- D2 pad 1: Net-(D3-K1) -> Net-(D2-K1)
- D2 pad 3: Net-(D3-K2) -> Net-(D2-K2)
- J14 pad 24: +5V-2 -> +12V-2
- J6 pad 24: +5V -> +12V
- NT1 pad 1: GND -> Net-(U5-OUT)
- NT1 pad 2: Net-(U13-Y2) -> Net-(U3A--)
- Q17 pad 1: Net-(Q5-B) (its old number) -> Net-(Q17-B)
- Q17 pad 2: GND-2 -> Net-(Q17-E)
- Q17 pad 3: Net-(Q5-C) (its old number) -> Net-(Q17-C)
- Q3 pad 1: Net-(Q2-B) -> Net-(Q3-B)
- Q3 pad 2: +5V-2 -> +12V-2
- Q4 pad 1: Net-(Q3-B) -> Net-(Q4-B)
- Q4 pad 2: +5V-2 -> +12V-2
- R1 pad 1: Net-(Q3-B) -> /Gate 1 x
- R1 pad 2: +5V-2 -> Net-(Q2-B)
- R26 pad 1: Net-(U2B--) -> /Note 1 Out
- R26 pad 2: Net-(U6-W) -> Net-(R26-Pad2)
- R27 pad 1: Net-(U2D--) -> Net-(U8B--)
- R29 pad 1: Net-(R42-Pad1) -> Net-(R29-Pad1)
- R3 pad 1: Net-(D4-K1) -> Net-(Q3-B)
- R3 pad 2: /Indicator 2 x -> Net-(Q1-C)
- R31 pad 1: Net-(U2D--) -> Net-(U8B--)
- R32 pad 2: Net-(U2D--) -> Net-(U8B--)
- R33 pad 2: Net-(U2C--) -> Net-(U8A--)
- R34 pad 1: Net-(R41-Pad1) -> Net-(R34-Pad1)
- R36 pad 1: DGND -> Net-(Q8-B)
- R36 pad 2: Net-(U13-Y) -> /Portament En
- R39 pad 2: Net-(C10-Pad2) (its old number) -> Net-(U10A-+)
- R4 pad 1: Net-(Q3-B) -> Net-(Q4-B)
- R4 pad 2: /Gate 1 x -> Net-(Q2-C)
- R41 pad 2: Net-(U2C--) -> Net-(U8A--)
- R42 pad 1: Net-(U2C--) -> Net-(U8A--)
- R44 pad 1: Net-(U10-A) -> Net-(Q10-S)
- R44 pad 2: /Gate 2 -> Net-(C37-Pad1)
- R45 pad 1: -12V -> /Velocity 2
- R45 pad 2: Net-(U10-W) -> Net-(Q10-S)
- R49 pad 1: Net-(U3C--) (its old number) -> Net-(C37-Pad1)
- R49 pad 2: Net-(U10-A) -> Net-(U13D--)
- R51 pad 2: Net-(C15-Pad2) (its old number) -> Net-(U10B-+)
- R52 pad 1: Net-(C10-Pad2) (its old number) -> /Velocity 1
- R52 pad 2: Net-(U2A--) -> Net-(Q11-S)
- R56 pad 1: Net-(U2A--) -> Net-(Q11-S)
- R56 pad 2: Net-(U5-W) -> Net-(C38-Pad1)
- R59 pad 1: Net-(U3B--) (its old number) -> Net-(C38-Pad1)
- R59 pad 2: Net-(U11-A) -> Net-(U13A--)
- R6 pad 1: Net-(D3-K1) -> Net-(D2-K2)
- R6 pad 2: /Indicator 1 x -> Net-(Q13-C)
- R60 pad 1: Net-(U10-A) -> Net-(U13D--)
- R63 pad 1: Net-(U11-A) -> Net-(U13A--)
- R69 pad 1: Net-(Q2-B) -> Net-(Q15-C)
- R69 pad 2: /Gate 2x -> Net-(D1-K1)
- R7 pad 2: Net-(D3-K2) -> Net-(D2-K1)
- R71 pad 1: Net-(Q5-C) (its old number) -> Net-(D1-K2)
- R71 pad 2: Net-(D4-K2) -> Net-(Q17-C)
- R73 pad 1: Net-(Q2-B) -> Net-(Q17-B)
- R73 pad 2: +5V-2 -> Net-(Q15-C)
- R77 pad 1: Net-(Q5-B) (its old number) -> Net-(Q17-B)
- R78 pad 1: /Indicator 2 x -> Net-(Q15-B)
- R78 pad 2: Net-(Q5-B) (its old number) -> GND-2
- R83 pad 1: /Gate 1 -> +12V
- R83 pad 2: Net-(U11-A) -> +A12V
- R84 pad 2: Net-(U11-W) -> -A12V
- U10 pad 1: Net-(U5-W) -> Net-(Q12-D)
- U10 pad 10: GND -> Net-(Q9-S)
- U10 pad 11: -12V -> GND
- U10 pad 12: GND -> Net-(Q12-S)
- U10 pad 13: Net-(U2D--) -> Net-(U10D--)
- U10 pad 14: Net-(R42-Pad1) -> Net-(U10D--)
- U10 pad 2: Net-(U2A--) -> Net-(Q12-D)
- U10 pad 3: GND -> Net-(U10A-+)
- U10 pad 4: +12V -> +A5V
- U10 pad 5: GND -> Net-(U10B-+)
- U10 pad 6: Net-(U2B--) -> Net-(Q9-D)
- U10 pad 7: Net-(U6-W) -> Net-(Q9-D)
- U10 pad 8: Net-(R41-Pad1) -> Net-(U10C--)
- U10 pad 9: Net-(U2C--) -> Net-(U10C--)
- U12 pad 1: +5V -> +A5V
- U12 pad 2: DGND -> GND
- U12 pad 4: Net-(U5-W) -> Net-(U10D--)
- U13 pad 10: /Velocity 2 -> GND
- U13 pad 11: -12V -> -A12V
- U13 pad 13: Net-(U10-A) -> Net-(U13D--)
- U13 pad 2: Net-(U11-A) -> Net-(U13A--)
- U13 pad 4: +12V -> +A12V
- U13 pad 5: /Velocity 1 -> GND
- U13 pad 6: Net-(U3B--) (its old number) -> Net-(Q11-S)
- U13 pad 7: Net-(U3B--) (its old number) -> Net-(C38-Pad1)
- U13 pad 8: Net-(U3C--) (its old number) -> Net-(C37-Pad1)
- U13 pad 9: Net-(U3C--) (its old number) -> Net-(Q10-S)
- U3 pad 11: -12V -> -A12V
- U3 pad 2: Net-(U13-X) -> Net-(U3A--)
- U3 pad 3: Net-(U13-Y) -> Net-(D5-A)
- U3 pad 4: +12V -> +A12V
- U3 pad 5: Net-(U7B-+) -> GND
- U4 pad 10: /CAN Rx -> /CAN Tx
- U4 pad 15: /Adjust S1 -> /Portament En
- U4 pad 33: /Resistor V2 -> /Resistor P2
- U4 pad 34: /Resistor V1 -> /Resistor P1
- U4 pad 9: /CAN Tx -> /CAN Rx
- U5 pad 1: +5V -> +A5V
- U5 pad 2: Net-(U12-OUT) -> Net-(U5-OUT)
- U6 pad 1: +5V -> Net-(D5-A)
- U6 pad 2: DGND -> Net-(R26-Pad2)
- U6 pad 3: Net-(U11-A) -> GND
- U6 pad 4: Net-(U11-W) -> +A12V
- U6 pad 5: /Resistor V1 -> +5V
- U6 pad 6: unconnected-(U11-B-Pad6) -> /Adjust S0
- U6 pad 7: unconnected-(U11-NC-Pad7) -> GND
- U6 pad 8: /Resistor U/D -> Net-(R28-Pad1)
- U7 pad 1: +5V -> +A5V
- U7 pad 2: DGND -> GND
- U7 pad 4: Net-(U6-W) -> Net-(U10C--)
Routing:
- net -12V: track 197.5 -> 6.99 mm, vias 6 -> 0
- net DGND: track 402.5 -> 231.3 mm, vias 2 -> 0
- net +A5V: track 0.00 -> 135.9 mm, vias 0 -> 7
- net +A12V: track 0.00 -> 121.5 mm, vias 0 -> 5
- net -A12V: track 0.00 -> 112.6 mm, vias 0 -> 8
- net +5V: track 338.3 -> 240.5 mm, vias 8 -> 2
- net GND: track 379.6 -> 462.3 mm, vias 5 -> 15
- net /Resistor P1: track 0.00 -> 75.2 mm, vias 0 -> 5
- net +12V: track 151.0 -> 78.4 mm, vias 6 -> 0
- net /Resistor V1: track 71.0 -> 0.00 mm, vias 5 -> 0
- net /Resistor V2: track 62.0 -> 0.00 mm, vias 3 -> 0
- net GND-2: track 94.4 -> 156.0 mm
- net /Adjust S1: track 59.2 -> 0.00 mm, vias 2 -> 0
- net /Resistor U/D: track 135.6 -> 90.4 mm
- net /Portament En: track 0.00 -> 43.7 mm, vias 0 -> 1
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Other:
- board text added: "CV Fountain"
- board text removed: "MIDI Decoder"
