File: kicad/midi_decoder.kicad_sch (KiCad schematic)
At the start: 153 parts, among them J10 Modulation CV, J11 CAN, J12 Bus Connector, J13 bus (board), J14 MIDI, J15 bus (controller), J2 MIDI, J3 MIDI IN, J4 MIDI THRU, J5 Note 1, J6 Gate 1, J7 Note 2, J8 Gate 2, J9 Expression CV, Q1 MMBT3906, Q2 MMBT3906, Q3 MMBT3906, Q4 MMBT3904, Q5 MMBT3904, Q6 MMBT3904, Q7 MMBT3904, SW1 Reset, U1 PEL12D-4225S-S2024, U10 TL074, U11 CD4052B, U12 REF3030, U13 MCP4011-103E/SN, U2 6N138, U3 SN65HVD1050D, U4 MCP4011-503E/SN, U5 TL074, U6 MCP4011-503E/SN, U7 MCP4011-103E/SN, U9 TL074, Y1 ECS-240-9

Commit message: revision 1
Parts:
- removed C11, C12, C15, C3: 0.1u, Capacitor_SMD:C_0805_2012Metric_Pad1.18x1.45mm_HandSolder, symbol Device:C_Small
- removed C17: 47p, Capacitor_SMD:C_0805_2012Metric_Pad1.18x1.45mm_HandSolder, symbol Device:C_Small
- removed D4: 1N4148, Diode_THT:D_DO-35_SOD27_P7.62mm_Horizontal, symbol Diode:1N4148
- removed NT1: NetTie_2, NetTie:NetTie-2_SMD_Pad0.5mm, symbol Device:NetTie_2
- removed Q1: MMBT3906, Package_TO_SOT_SMD:SOT-23, symbol Transistor_BJT:MMBT3906
- removed Q7: MMBT3904, Package_TO_SOT_SMD:SOT-23, symbol Transistor_BJT:MMBT3904
- removed R20: 330k, Resistor_SMD:R_0805_2012Metric_Pad1.20x1.40mm_HandSolder, symbol Device:R_Small_US
- removed R21, R32: 270k, Resistor_SMD:R_0805_2012Metric_Pad1.20x1.40mm_HandSolder, symbol Device:R_Small_US
- removed R33, R34: 470k, Diode_SMD:D_0805_2012Metric_Pad1.15x1.40mm_HandSolder, symbol Device:R_Small_US
- removed R35: 1meg, Diode_SMD:D_0805_2012Metric_Pad1.15x1.40mm_HandSolder, symbol Device:R_Small_US
- removed R39: 4.7meg, Diode_SMD:D_0805_2012Metric_Pad1.15x1.40mm_HandSolder, symbol Device:R_Small_US
- removed R42: 470k 1%, Diode_SMD:D_0805_2012Metric_Pad1.15x1.40mm_HandSolder, symbol Device:R_Small_US
- removed R5, R6, R75: 10k, Diode_SMD:D_0805_2012Metric_Pad1.15x1.40mm_HandSolder, symbol Device:R_Small_US
- removed U11: CD4052B, Package_SO:SOIC-16_3.9x9.9mm_P1.27mm, symbol Analog_Switch:CD4052B
- removed U4, U6: MCP4011-503E/SN, Package_SO:SOIC-8_3.9x4.9mm_P1.27mm, symbol Potentiometer_Digital:MCP4011-xxxxSN
- removed Y1: ECS-240-9, Crystal:Crystal_SMD_3225-4Pin_3.2x2.5mm_HandSoldering, symbol Device:Crystal_GND24
- added C14, C21: 4.7u tantal, Capacitor_Tantalum_SMD:CP_EIA-3216-10_Kemet-I_Pad1.58x1.35mm_HandSolder, symbol Device:C_Polarized_Small
- added C16, C17: 100u, Capacitor_SMD:CP_Elec_5x5.3, symbol Device:C_Polarized_Small
- added C18, C22: 100u, Capacitor_THT:CP_Radial_D6.3mm_P2.50mm, symbol Device:C_Polarized_Small
- added C31, C32, C33, C9: 0.1u, Capacitor_SMD:C_0805_2012Metric_Pad1.18x1.45mm_HandSolder, symbol Device:C_Small
- added C37, C38: 56p, Capacitor_SMD:C_0805_2012Metric_Pad1.18x1.45mm_HandSolder, symbol Device:C_Small
- added D4, D5, D6, D7: 1N4448WS, Diode_SMD:D_SOD-323_HandSoldering, symbol Diode:1N4448WS
- added L1: 22u, Inductor_SMD:L_0805_2012Metric_Pad1.05x1.20mm_HandSolder, symbol Device:L_Small
- added Q1, Q13, Q15, Q16, Q17, Q18, Q2: BC847B, Package_TO_SOT_SMD:SOT-23, symbol Transistor_BJT:MMBT3904
- added Q10, Q11: MMBFJ176, Package_TO_SOT_SMD:SOT-23, symbol JFET:MMBFJ176
- added Q12, Q9: MMBFJ112, Package_TO_SOT_SMD:SOT-23, symbol Transistor_FET:MMBFJ112
- added Q3, Q8: BC857B, Package_TO_SOT_SMD:SOT-23, symbol Transistor_BJT:MMBT3906
- added R22: 806k 1%, Diode_SMD:D_0805_2012Metric_Pad1.15x1.40mm_HandSolder, symbol Device:R_Small_US
- added R26, R40, R64: 220k, Diode_SMD:D_0805_2012Metric_Pad1.15x1.40mm_HandSolder, symbol Device:R_Small_US
- added R43, R44, R56, R57: 470k, Resistor_SMD:R_0805_2012Metric_Pad1.20x1.40mm_HandSolder, symbol Device:R_Small_US
- added R52: 200k, Resistor_SMD:R_0805_2012Metric_Pad1.20x1.40mm_HandSolder, symbol Device:R_Small_US
- added R54, R55: 100k, Resistor_SMD:R_0805_2012Metric_Pad1.20x1.40mm_HandSolder, symbol Device:R_Small_US
- added R58: 22k, Resistor_SMD:R_0805_2012Metric_Pad1.20x1.40mm_HandSolder, symbol Device:R_Small_US
- added R69, R71: 2.2k, Diode_SMD:D_0805_2012Metric_Pad1.15x1.40mm_HandSolder, symbol Device:R_Small_US
- added R72: 22k, Diode_SMD:D_0805_2012Metric_Pad1.15x1.40mm_HandSolder, symbol Device:R_Small_US
- added R74, R77: 47k, Diode_SMD:D_0805_2012Metric_Pad1.15x1.40mm_HandSolder, symbol Device:R_Small_US
- added R78: 10k, Diode_SMD:D_0805_2012Metric_Pad1.15x1.40mm_HandSolder, symbol Device:R_Small_US
- added R83, R84: 5, Resistor_SMD:R_0805_2012Metric_Pad1.20x1.40mm_HandSolder, symbol Device:R_Small_US
- added U14, U9: MCP4011-503E/SN, Package_SO:SOIC-8_3.9x4.9mm_P1.27mm, symbol Potentiometer_Digital:MCP4011-xxxxSN
- added U6: DG419LDY, Package_SO:SOIC-8_3.9x4.9mm_P1.27mm, symbol Analog_Switch:DG419LDY
- added U8: TL072, Package_SO:SOIC-8_3.9x4.9mm_P1.27mm, symbol Amplifier_Operational:TL072
- added XTAL1: ABM7-24.000MHZ-D2Y-T, MyCrystal:XTAL_ABM7_ABR_handsoldering, symbol Crystal:ABM7-24.000MHZ-D2Y-T
- C24: renamed from C29; value 8p -> 18p
- C25: renamed from C27; value 8p -> 18p
- C26: value 0.1u -> 56p
- D1: value Note 2 -> Note 1
- Q14: renamed from Q6; value MMBT3904 -> BC847B
- Q4: renamed from Q2; value MMBT3906 -> BC857B
- Q5: renamed from Q4; value MMBT3904 -> BC847B
- Q6: renamed from Q3; value MMBT3906 -> BC857B
- Q7: renamed from Q5; value MMBT3904 -> BC847B
- R14: renamed from R63; value 10k -> 22k
- R17: renamed from R38; value 10k -> 100k
- R2: value 1k -> 10k
- R20: renamed from R37; value 10k -> 22k
- R23: renamed from R43; value 470k -> 470k 1%
- R24: renamed from R41; value 470k -> 500k 1%
- R27: renamed from R55; value 150k 1% -> 200k 0.1%
- R28: value 330k -> 220k; footprint Resistor_SMD:R_0805_2012Metric_Pad1.20x1.40mm_HandSolder -> Diode_SMD:D_0805_2012Metric_Pad1.15x1.40mm_HandSolder
- R3: value 220 -> 10k
- R31: renamed from R48; value 145k 1% -> 200k 0.1%
- R32: renamed from R54; value 145k -> 95.3k
- R33: renamed from R49; value 145k 1% -> 200k 0.1%
- R35: renamed from R40; value 10k -> 10k 1%
- R36: value 1meg -> 10k
- R37: renamed from R46; value 10k -> 10k 1%
- R38: renamed from R44; value 10k -> 10k 1%
- R41: renamed from R53; value 145k -> 95.3k
- R42: renamed from R51; value 150k 1% -> 200k 0.1%
- R45: value 470k 1% -> 200k; footprint Diode_SMD:D_0805_2012Metric_Pad1.15x1.40mm_HandSolder -> Resistor_SMD:R_0805_2012Metric_Pad1.20x1.40mm_HandSolder
- R47: value 4.7meg -> 22k; footprint Diode_SMD:D_0805_2012Metric_Pad1.15x1.40mm_HandSolder -> Resistor_SMD:R_0805_2012Metric_Pad1.20x1.40mm_HandSolder
- R6: renamed from R9; value 1k -> 2.2k
- R60: renamed from R31; value 200k -> 100k
- R63: renamed from R18; value 200k -> 100k
- R7: renamed from R8; value 220 -> 2.2k
- R73: value 10k -> 220k
- U10: renamed from U9; value TL074 -> LMV324A
- renumbered C22 to C1, C1 to C11, C7 to C12, C6 to C13, C5 to C15, C2 to C19, C21 to C2, C31 to C23, C24 to C27, C13 to C28, C25 to C29, C18 to C3, C16 to C30, C30 to C34, C28 to C35, C23 to C36, C14 to C4, C8 to C5, C19 to C6, C9 to C7, C4 to C8, D3 to D2, D2 to D3, H2 to H1, H1 to H2, J4 to J1, J8 to J10, J10 to J12, J12 to J13, J15 to J14, J3 to J2, J2 to J3, J14 to J4, J13 to J6, J6 to J8, NT2 to NT1, R14 to R11, R16 to R12, R15 to R13, R7 to R15, R59 to R16, R56 to R18, R57 to R19, R58 to R21, R60 to R25, R50 to R29, R61 to R30, R52 to R34, R29 to R39, R27 to R46, R26 to R48, R25 to R49, R13 to R5, R24 to R50, R23 to R51, R30 to R53, R19 to R59, R22 to R61, R17 to R62, R62 to R65, R67 to R66, R64 to R67, R65 to R68, R74 to R70, R72 to R75, R66 to R76, R68 to R79, R11 to R8, R69 to R80, R70 to R81, R71 to R82, R12 to R9, U3 to U11, U13 to U12, U5 to U13, U10 to U3, U8 to U4, U12 to U5
Connections:
- net +12V: now also J6.24 (Pin_24), R83.1; no longer C27.1, C29.1, C34.1, U10.4 (V+), U13.4 (V+), U3.4 (V+)
- net +5V: now also C17.1, L1.1, U6.5 (VL); no longer C20.1, C30.2, C36.2, J6.24 (Pin_24), R45.2, U12.1 (VDD), U5.1 (IN), U7.1 (VDD)
- net -12V: now also R84.1; no longer C26.2, C28.2, C35.2, U10.11 (V-), U13.11 (V-), U3.11 (V-)
- net Adjust En: now also D5.1 (K)
- net Adjust S0: now also U6.6
- net Bend Out: now also C26.1
- net CAN Rx: now also U4.9 (P12_7(UART_TX)); no longer U4.10 (P12_6(UART_RX))
- net CAN Tx: now also U4.10 (P12_6(UART_RX)); no longer U4.9 (P12_7(UART_TX))
- net DGND: now also D4.2 (A); no longer C20.2, C30.1, C36.1, R47.1, U12.2 (VSS), U7.2 (VSS)
- net GND: now also C20.1, C30.1, C36.1, R47.1, U10.11 (V-), U12.2 (VSS), U13.10 (+), U13.5 (+), U3.5 (+), U7.2 (VSS), C14.2, C16.2, C17.2, C18.2, C21.2, C22.1, C31.1, C32.2, C33.2, C9.1, R58.1, U14.2 (VSS), U6.3 (GND), U6.7 (V-), U8.3 (+), U8.5 (+), U9.2 (VSS); no longer C26.1, U10.10 (+), U10.12 (+), U10.3 (+), U10.5 (+)
- net GND-2: now also Q1.2 (E), Q13.2 (E), Q15.2 (E), Q18.2 (E), Q2.2 (E), R74.2, R77.2, R78.2; no longer R73.2
- net Gate 1: now also Q11.3 (G)
- net Gate 1 x: now also R1.1; no longer R4.2
- net Gate 2: now also Q10.3 (G); no longer R28.2
- net Gate 2x: now also R2.1
- net Indicator 1 x: no longer R6.2
- net Indicator 2 x: now also R72.1; no longer R2.2
- net Note 1 Out: now also R26.1
- net Note 2 Out: now also R28.2
- net Resistor U/D: now also U14.8 (U/~{D}), U9.8 (U/~{D})
- net Velocity 1: now also R52.1; no longer U13.5 (+)
- net Velocity 2: now also R45.1; no longer U13.10 (+)
- net at U12.4 (W): now also U10.13 (-), U10.14; no longer U10.1
- net at R33.2, R41.2, R42.1: now also U8.2 (-); no longer U10.9 (-)
- net at C25.1, U4.42 (P15_1): now also XTAL1.2
- net at C8.2, R51.2: now also U10.5 (+)
- net at R36.1: now also Q8.1 (B); no longer U10.6 (-)
- net at U3.2 (-): now also NT1.2
- net at U10.2 (-): now also U10.1, Q12.1 (D), U14.6 (B)
- net at Q7.1 (B), R17.2, R20.2: now also D4.1 (K)
- net at R23.2, R24.1, U3.6 (-): now also C26.2, R22.1
- net at Q4.1 (B), R4.1: no longer R1.1
- net at R73.1: now also Q17.1 (B), R77.1
- net at R59.1, U13.7: now also C38.1, R56.2; no longer U13.6 (-)
- net at Q14.3 (C), R7.1: now also R64.2
- net at R7.2: now also D2.1 (K1); no longer D2.3 (K2)
- net at R49.2, R60.1, U13.13 (-): no longer R28.1
- net at R47.2: now also R43.2, R54.1; no longer U3.3 (+)
- net at C24.1, U4.43 (P15_0): now also XTAL1.1
- net at R29.1: now also U8.7; no longer U10.14
- net at D1.2 (A): now also Q3.3 (C)
- net at R27.1, R31.1, R32.2: now also U8.6 (-); no longer U10.13 (-)
- net at R49.1, U13.8: now also C37.1, R44.2; no longer U13.9 (-)
- net at R3.1: now also Q3.1 (B)
- net at D1.3 (K2): now also R71.1; no longer R3.2
- net at C5.2, R39.2: now also U10.3 (+)
- net at U10.8: now also U10.9 (-), U7.4 (W); no longer R34.1
- net at D1.1 (K1): now also R69.2; no longer R2.1
- net at R6.1: now also D2.3 (K2); no longer D2.1 (K1)
- net +5V-2 renamed +12V-2
- net +12V-2: now also Q3.2 (E); no longer R1.2
- net Adjust S1 renamed Portament En
- net Portament En: now also R36.2
- net Resistor V1 renamed Resistor P1
- net Resistor P1: now also U14.5 (~{CS})
- net Resistor V2 renamed Resistor P2
- net Resistor P2: now also U9.5 (~{CS})
- new net: C37.2, Q10.2 (S), R44.1, R45.2, U13.9 (-)
- new net: Q1.3 (C), R3.2
- new net: R28.1, U6.8
- new net: Q11.1 (D), R57.1
- new net: C38.2, Q11.2 (S), R52.2, R56.1, U13.6 (-)
- new net: Q2.1 (B), R1.2
- new net: R26.2, U6.2
- new net: Q15.1 (B), R72.2, R78.1
- new net: D6.1 (K), D7.1 (K), Q8.3 (C), R40.2
- new net: D6.2 (A), Q9.3 (G)
- new net: Q10.1 (D), R43.1
- new net: Q17.2 (E), Q18.1 (B)
- new net: Q17.3 (C), Q18.3 (C), R71.2
- new net: D7.2 (A), Q12.3 (G)
- new net: Q15.3 (C), R69.1, R73.2
- new net: Q1.1 (B), R2.2
- new net: Q16.1 (B), R64.1, R74.1
- new net: D5.2 (A), U3.3 (+), U6.1
- new net: C21.1, U14.4 (W)
- new net: Q12.2 (S), U10.12 (+), U14.3 (A)
- new net: R55.1, R57.2, R58.2
- new net: Q9.1 (D), U10.6 (-), U10.7, U9.6 (B)
- new net: Q2.3 (C), R4.2
- new net: Q9.2 (S), U10.10 (+), U9.3 (A)
- new net: R34.1, U8.1
- new net: Q13.1 (B), Q16.2 (E)
- new net: Q13.3 (C), Q16.3 (C), R6.2
- new net: C14.1, U9.4 (W)
- new net +A12V: C18.1, C27.1, C32.1, C33.1, C34.1, R22.2, R83.2, U13.4 (V+), U3.4 (V+), U6.4 (V+), U8.8 (V+)
- new net +A5V: C16.1, C20.2, C29.1, C30.2, C36.2, C9.2, L1.2, Q8.2 (E), U10.4 (V+), U12.1 (VDD), U14.1 (VDD), U5.1 (IN), U7.1 (VDD), U9.1 (VDD)
- new net -A12V: C22.2, C28.2, C31.2, C35.2, R40.1, R54.2, R55.2, R84.2, U13.11 (V-), U3.11 (V-), U8.4 (V-)
- no-connect marks 42 -> 40
Other:
- note removed: "Velo_1 offset"
- note removed: "Velo_2 offset"
- moved on the sheet: C1, C10, C12, C13, C15, C27, C28, C29, C3, C30, C34, C35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
