File: kicad/cv-depot.kicad_sch (KiCad schematic)
At the start: 184 parts, among them J1 MIDI THRU, J10 Gate 2, J11 CAN, J12 Modulation CV, J13 Bus Connector, J14 bus (controller), J2 MIDI IN, J3 MIDI, J4 MIDI, J5 Note 1, J6 bus (board), J7 Note 2, J8 Gate 1, J9 Expression CV, Q1 BC847B, Q10 MMBFJ176, Q11 MMBFJ176, Q12 MMBFJ112, Q13 BC847B, Q14 BC847B, Q15 BC847B, Q16 BC847B, Q17 BC847B, Q18 BC847B, Q2 BC847B, Q3 BC857B, Q4 BC857B, Q5 BC847B, Q6 BC857B, Q7 BC847B, Q8 BC857B, Q9 MMBFJ112, SW1 Reset, U1 PEL12D-4225S-S2024, U10 LMV324A, U11 SN65HVD1050D, U12 MCP4011-103E/SN, U13 TL074, U14 MCP4011-503E/SN, U2 6N138, U3 TL074, U5 REF3030, U6 DG419LDY, U7 MCP4011-103E/SN, U8 TL072, U9 MCP4011-503E/SN

Commit message: done with initial hardware check except voltage outputs
Parts:
- R6, R69, R7, R71: value 2.2k -> 1k
- R75: value 220 -> 470
Changed lines of the file:
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@@
 			)
 		)
-		(property "Value" "2.2k"
+		(property "Value" "1k"
 			(at 105.41 116.84 90)
 			(effects
@@
 			)
 		)
-		(property "Value" "2.2k"
+		(property "Value" "1k"
 			(at 101.854 138.938 90)
 			(effects
@@
 			)
 		)
-		(property "Value" "220"
+		(property "Value" "470"
 			(at 90.17 196.85 90)
 			(effects
@@
 			)
 		)
-		(property "Value" "2.2k"
+		(property "Value" "1k"
 			(at 105.664 95.758 90)
 			(effects
@@
 			)
 		)
-		(property "Value" "2.2k"
+		(property "Value" "1k"
 			(at 101.6 160.02 90)
 			(effects

Commit message: added digital pot controller, verified in debugger (not yet in full speed)
Connections:
- net Resistor N1 renamed Pot N1
- net Resistor N2 renamed Pot N2
- net Resistor P1 renamed Pot P1
- net Resistor P2 renamed Pot P2
- net Resistor U/D renamed Pot U/D
Changed lines of the file:
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@@
 		)
 	)
-	(label "Resistor P2"
+	(label "Pot P2"
 		(at 285.75 254 0)
 		(effects
@@
 		)
 	)
-	(label "Resistor U{slash}D"
+	(label "Pot U{slash}D"
 		(at 285.75 259.08 0)
 		(effects
@@
 		)
 	)
-	(label "Resistor P1"
+	(label "Pot P1"
 		(at 285.75 256.54 0)
 		(effects
@@
 		)
 	)
-	(label "Resistor N2"
+	(label "Pot N2"
 		(at 285.75 248.92 0)
 		(effects
@@
 		)
 	)
-	(label "Resistor N1"
+	(label "Pot N1"
 		(at 285.75 251.46 0)
 		(effects

Commit message: Modified the value of the resistor for the green LED
Parts:
- R75: value 470 -> 820
Changed lines of the file:
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@@
 			)
 		)
-		(property "Value" "470"
+		(property "Value" "820"
 			(at 90.17 196.85 90)
 			(effects
